File: scheme/doorbell.kicad_pcb (KiCad board)
At the start: 2 copper layers, 0 parts

Commit message: next step
Parts:
- added DD1: ATTINY45, DIP-8__300_ELL, F.Cu at (50.8, 41.3)
- added R1: RES, R4-5, F.Cu at (38.7, 29.8)
- added R2: RES, R4-5, F.Cu at (66.7, 26.7)
- added R3: RES_VAR, C1-1, F.Cu at (37.5, 52.7)
- added SF1: SF, AK300-2, F.Cu at (83.8, 35.6)
- added SP1: SPEAKER, C2, F.Cu at (59.1, 62.2)
- added VT1: КТ315, TO220_VERT, F.Cu at (42.5, 63.5)
- added XS1: Питание, AK300-2, F.Cu at (83.8, 49.5)
- added XS3: Кнопки, C2, F.Cu at (51.4, 25.4)

Commit message: next step
Parts:
- removed XS3: Кнопки, C2
- added R4: 100, R4-5, F.Cu at (87.6, 80.0)
- added SA1: SA, C2, F.Cu at (80.0, 68.6)
- added VD1: LED, C2, F.Cu at (88.9, 68.6)
- added VD2: LED, C2, F.Cu at (58.4, 68.6)
- added XS2: пуск, 1pinsmall, F.Cu at (64.8, 68.6)
- R1: value RES -> 5,1к
- R2: value RES -> 1к; footprint R4-5 -> RV2
- R3: value RES_VAR -> 100; footprint C1-1 -> R4-5
- SF1, XS1: footprint AK300-2 -> C2
- moved R1 67.4 mm to (83.8, 80.0), turned to 270 degrees
- moved R2 55.1 mm to (73.7, 81.3)
- moved R3 43.9 mm to (62.2, 88.9), turned to 180 degrees
- moved SF1 42.2 mm to (99.1, 74.9)
- moved XS1 41.0 mm to (99.1, 87.6)
- moved DD1 40.0 mm to (61.0, 80.0), turned to 270 degrees
- moved VT1 32.7 mm to (73.7, 73.7)
- moved SP1 13.6 mm to (71.1, 68.6)
Connections:
- DD1 pad 2: (no net) -> N-000008
- DD1 pad 6: N-000003 -> N-000002
- DD1 pad 7: N-000004 -> N-0000010
- R1 pad 1: N-000002 -> N-000001
- R1 pad 2: N-000003 -> N-000004
- R2 pad 1: N-000004 -> N-000002
- R2 pad 2: N-000001 -> GND
- R3 pad 1: N-000008 -> N-000009
- R3 pad 2: N-000002 -> N-000008
- SF1 pad 2: N-000001 -> N-000003
- VT1 pad 1: N-000008 -> N-000001
Other:
- board outline added: 50 x 25 mm

Commit message: small changes
Parts:
- DD1: footprint DIP-8__300_ELL -> dip8-soic
- R2: footprint RV2 -> res-var
- SF1, XS1: footprint C2 -> terminal-2pin
- VT1: footprint TO220_VERT -> kt315
- moved R2 5.06 mm to (75.2, 86.1)
- moved XS1 2.55 mm to (98.8, 85.1)
- moved VT1 1.44 mm to (74.7, 74.7), turned to 0 degrees
- moved SF1 1.05 mm to (98.8, 73.9)

Commit message: small changes
Parts:
- moved R1 17.7 mm to (77.5, 96.5), turned to 0 degrees
- moved R4 17.3 mm to (92.7, 96.5), turned to 180 degrees
- moved VT1 9.61 mm to (84.0, 77.0), turned to 270 degrees
- moved R3 7.73 mm to (61.0, 96.5)
- moved R2 6.22 mm to (74.0, 80.0)
- moved XS1 5.81 mm to (93.0, 85.0)
- moved SF1 5.81 mm to (93.0, 74.0)
- moved DD1 1.99 mm to (61.0, 82.0)
- moved VD1 0.59 mm to (89.0, 68.0)
Other:
- board size 50 x 25 mm -> 50 x 35 mm

Commit message: next step
Parts:
- added R5: 3,6к, R3, F.Cu at (85.0, 86.0)
- R1, R3, R4: footprint R4-5 -> R3
- SA1, SP1: footprint C2 -> SIL-2
- VD1: value LED -> красный; footprint C2 -> SIL-2
- VD2: value LED -> зеленый; footprint C2 -> SIL-2
- XS2: footprint 1pinsmall -> SIL-1
- moved R4 36.5 mm to (64.0, 74.0)
- moved VD1 32.6 mm to (56.4, 69.1)
- moved XS2 19.3 mm to (73.0, 86.0)
- moved R1 18.2 mm to (87.0, 81.0), turned to 180 degrees
- moved R3 17.1 mm to (54.4, 80.8), turned to 270 degrees
- moved SP1 12.1 mm to (83.0, 71.0)
- moved VD2 6.12 mm to (64.5, 69.1)
- moved SA1 6.02 mm to (74.0, 69.0)
- moved VT1 5.39 mm to (89.0, 75.0), turned to 90 degrees
- moved SF1 4.00 mm to (97.0, 74.0)
- moved XS1 4.00 mm to (97.0, 85.0)
- moved DD1 3.00 mm to (64.0, 82.0)
- moved R2 2.00 mm to (76.0, 80.0)
Routing:
- net GND: track 0.00 -> 124.8 mm
- net V+: track 0.00 -> 95.2 mm
- net N-000009: track 0.00 -> 23.6 mm
- net N-0000011: track 0.00 -> 14.2 mm
- net N-0000010: track 0.00 -> 13.4 mm
- net N-000004: track 0.00 -> 9.29 mm
- net N-000003: track 0.00 -> 8.93 mm
- net N-000007: track 0.00 -> 8.19 mm
- net N-000005: track 0.00 -> 7.75 mm
- net N-000002: track 0.00 -> 7.43 mm
- net N-0000012: track 0.00 -> 5.75 mm
- net N-000001: track 0.00 -> 4.64 mm
Other:
- board size 50 x 35 mm -> 50 x 26 mm

Commit message: small changes
Parts:
- added PIN_ARRAY_1: Val**, PIN_ARRAY_1, F.Cu at (77.0, 89.0)
- moved XS2 16.4 mm to (74.2, 69.6)
- moved SA1 9.86 mm to (83.8, 69.8)
- moved SP1 7.17 mm to (90.2, 70.9)
- moved R1 4.25 mm to (90.4, 78.5), turned to 270 degrees
- moved VT1 4.06 mm to (85.6, 77.2)
- moved R3 3.70 mm to (55.4, 77.2)
- moved R5 1.65 mm to (86.6, 86.4)
- moved R4 1.36 mm to (64.0, 72.6)
- moved VD1 1.27 mm to (57.7, 69.1)
- moved SF1 1.23 mm to (97.5, 72.9)
- moved XS1 0.86 mm to (97.5, 84.3), turned to 270 degrees
- moved VD2 0.76 mm to (65.3, 69.1)
- moved R2 0.67 mm to (76.5, 79.5)
- moved DD1 0.38 mm to (63.8, 82.3)
Routing:
- net (no net): track 0.00 -> 150.0 mm
- net N-0000010: track 13.4 -> 41.6 mm
- net N-000009: track 23.6 -> 14.0 mm
- net N-0000011: track 14.2 -> 23.4 mm
- net N-000001: track 4.64 -> 12.2 mm
- net V+: track 95.2 -> 100.3 mm
- net N-000004: track 9.29 -> 4.83 mm
- net N-000003: track 8.93 -> 13.3 mm
- net GND: track 124.8 -> 121.0 mm
- net N-000007: track 8.19 -> 4.74 mm
- net N-000002: track 7.43 -> 4.57 mm
- net N-0000012: track 5.75 -> 4.08 mm
- net N-000005: track 7.75 -> 8.78 mm
Other:
- board size 50 x 26 mm -> 50 x 25 mm

Commit message: small changes
Parts:
- moved SA1 1.78 mm to (82.0, 69.8)
- moved SF1 1.61 mm to (96.0, 73.4)
- moved XS1 1.52 mm to (96.0, 84.3)
- moved SP1 1.27 mm to (88.9, 70.9)
Routing:
- net GND: track 121.0 -> 115.9 mm
- net N-0000011: track 23.4 -> 22.4 mm
- net V+: track 100.3 -> 101.1 mm
- net N-000009: track 14.0 -> 14.6 mm
- net N-000003: track 13.3 -> 12.8 mm
Changed lines of the file:
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@@
   )
   (setup
-    (last_trace_width 0.254)
+    (last_trace_width 1)
     (user_trace_width 0.5)
     (user_trace_width 1)
@@
   )
   (module terminal-2pin (layer F.Cu)
-    (at 97.536 72.898 90)
+    (at 96.012 73.406 90)
     (descr "Condensateur = 2 pas")
     (tags C)
@@
   )
   (module terminal-2pin (layer F.Cu)
-    (at 97.536 84.328 270)
+    (at 96.012 84.328 270)
     (descr "Condensateur = 2 pas")
     (tags C)
@@
   )
   (module SIL-2 (layer F.Cu)
-    (at 90.17 70.866 180)
+    (at 88.9 70.866 180)
     (descr "Connecteurs 2 pins")
     (tags "CONN DEV")
@@
   )
   (module SIL-2 (layer F.Cu)
-    (at 83.82 69.85 180)
+    (at 82.042 69.85 180)
     (descr "Connecteurs 2 pins")
     (tags "CONN DEV")
@@
   (segment (start 52 91) (end 102 91) (width 0.254) (layer B.Cu) (net 0))
   (segment (start 59.944 86.106) (end 60.198 86.106) (width 0.5) (layer B.Cu) (net 1))
-  (segment (start 94.996 89.408) (end 97.536 86.868) (width 1) (layer B.Cu) (net 1))
+  (segment (start 94.996 89.408) (end 96.012 86.868) (width 1) (layer B.Cu) (net 1) (status 20))
   (segment (start 82.296 89.408) (end 94.996 89.408) (width 1) (layer B.Cu) (net 1))
-  (segment (start 79.248 86.36) (end 82.296 89.408) (width 1) (layer B.Cu) (net 1))
-  (segment (start 74.422 86.36) (end 79.248 86.36) (width 1) (layer B.Cu) (net 1))
-  (segment (start 72.136 88.646) (end 74.422 86.36) (width 1) (layer B.Cu) (net 1))
+  (segment (start 79.248 86.614) (end 82.296 89.408) (width 1) (layer B.Cu) (net 1))
+  (segment (start 74.422 86.614) (end 79.248 86.614) (width 1) (layer B.Cu) (net 1))
+  (segment (start 72.136 88.646) (end 74.422 86.614) (width 1) (layer B.Cu) (net 1))
   (segment (start 62.738 88.646) (end 72.136 88.646) (width 1) (layer B.Cu) (net 1))
   (segment (start 60.198 86.106) (end 62.738 88.646) (width 1) (layer B.Cu) (net 1))
   (segment (start 77.04 81.646) (end 77.836 81.646) (width 1) (layer B.Cu) (net 1))
   (segment (start 86.868 86.36) (end 90.424 86.36) (width 1) (layer B.Cu) (net 1))
-  (segment (start 84.074 83.566) (end 86.868 86.36) (width 1) (layer B.Cu) (net 1))
-  (segment (start 79.756 83.566) (end 84.074 83.566) (width 1) (layer B.Cu) (net 1))
+  (segment (start 84.074 84.074) (end 86.868 86.36) (width 1) (layer B.Cu) (net 1))
+  (segment (start 79.756 83.566) (end 84.074 84.074) (width 1) (layer B.Cu) (net 1))
   (segment (start 77.836 81.646) (end 79.756 83.566) (width 1) (layer B.Cu) (net 1))
-  (segment (start 97.536 86.868) (end 93.218 86.868) (width 1) (layer B.Cu) (net 1))
+  (segment (start 96.012 86.868) (end 93.218 86.868) (width 1) (layer B.Cu) (net 1) (status 10))
   (segment (start 91.186 86.36) (end 90.424 86.36) (width 0.5) (layer B.Cu) (net 1) (status 30))
   (segment (start 93.218 86.868) (end 91.186 86.36) (width 1) (layer B.Cu) (net 1) (status 20))
   (segment (start 85.598 79.756) (end 89.154 79.756) (width 1) (layer B.Cu) (net 1))
-  (segment (start 90.932 77.978) (end 94.488 77.978) (width 1) (layer B.Cu) (net 1))
+  (segment (start 90.932 77.978) (end 93.218 77.978) (width 1) (layer B.Cu) (net 1))
   (segment (start 89.154 79.756) (end 90.932 77.978) (width 1) (layer B.Cu) (net 1))
   (segment (start 58.928 69.088) (end 58.928 70.612) (width 1) (layer B.Cu) (net 1))
@@
   (segment (start 57.658 71.882) (end 57.658 77.47) (width 1) (layer B.Cu) (net 1))
   (segment (start 58.928 70.612) (end 57.658 71.882) (width 1) (layer B.Cu) (net 1))
-  (segment (start 97.536 86.868) (end 94.488 83.82) (width 1) (layer B.Cu) (net 1))
-  (segment (start 94.488 83.82) (end 94.488 77.978) (width 1) (layer B.Cu) (net 1))
-  (segment (start 97.028 75.438) (end 97.536 75.438) (width 0.5) (layer B.Cu) (net 1))
-  (segment (start 94.488 77.978) (end 97.028 75.438) (width 1) (layer B.Cu) (net 1))
+  (segment (start 96.012 86.868) (end 93.218 83.312) (width 1) (layer B.Cu) (net 1) (status 400010))
+  (segment (start 93.218 83.312) (end 93.218 77.978) (width 1) (layer B.Cu) (net 1))
+  (segment (start 95.504 75.946) (end 96.012 75.946) (width 0.5) (layer B.Cu) (net 1) (status 30))
+  (segment (start 93.218 77.978) (end 95.504 75.946) (width 1) (layer B.Cu) (net 1) (status 20))
   (segment (start 58.928 69.088) (end 64.008 69.088) (width 1) (layer B.Cu) (net 1) (status 20))
   (segment (start 90.424 82.296) (end 82.804 82.296) (width 0.5) (layer B.Cu) (net 2))
@@
   (segment (start 82.804 82.296) (end 79.614 79.106) (width 0.5) (layer B.Cu) (net 2))
   (segment (start 67.564 86.106) (end 71.374 86.106) (width 0.5) (layer B.Cu) (net 3))
-  (segment (start 81.28 84.836) (end 82.804 86.36) (width 0.5) (layer B.Cu) (net 3))
-  (segment (start 72.644 84.836) (end 81.28 84.836) (width 0.5) (layer B.Cu) (net 3))
+  (segment (start 82.042 85.344) (end 82.804 86.36) (width 0.5) (layer B.Cu) (net 3))
+  (segment (start 72.644 84.836) (end 82.042 85.344) (width 0.5) (layer B.Cu) (net 3))
   (segment (start 71.374 86.106) (end 72.644 84.836) (width 0.5) (layer B.Cu) (net 3))
   (segment (start 65.024 76.454) (end 69.088 76.454) (width 0.5) (layer B.Cu) (net 3))
   (segment (start 65.024 86.106) (end 65.024 76.454) (width 0.5) (layer B.Cu) (net 3))
   (segment (start 67.564 86.106) (end 65.024 86.106) (width 0.5) (layer B.Cu) (net 3))
-  (segment (start 74.168 71.374) (end 74.168 69.596) (width 0.5) (layer B.Cu) (net 3) (status 800020))
+  (segment (start 74.168 71.374) (end 74.168 69.596) (width 0.5) (layer B.Cu) (net 3) (status 20))
   (segment (start 70.358 75.438) (end 74.168 71.374) (width 0.5) (layer B.Cu) (net 3))
   (segment (start 69.088 76.454) (end 70.358 75.438) (width 0.5) (layer B.Cu) (net 3))
   (segment (start 67.564 81.026) (end 69.85 81.026) (width 0.5) (layer B.Cu) (net 4))
-  (segment (start 81.28 70.104) (end 82.55 69.85) (width 0.5) (layer B.Cu) (net 4) (status 20))
-  (segment (start 81.28 75.946) (end 81.28 70.104) (width 0.5) (layer B.Cu) (net 4))
+  (segment (start 81.28 71.374) (end 80.772 69.85) (width 0.5) (layer B.Cu) (net 4) (status 20))
+  (segment (start 81.28 75.946) (end 81.28 71.374) (width 0.5) (layer B.Cu) (net 4))
   (segment (start 81.026 76.2) (end 81.28 75.946) (width 0.5) (layer B.Cu) (net 4))
   (segment (start 73.914 76.2) (end 81.026 76.2) (width 0.5) (layer B.Cu) (net 4))
@@
   (segment (start 55.372 81.026) (end 59.944 81.026) (width 0.5) (layer B.Cu) (net 6))
   (segment (start 85.598 77.216) (end 84.582 77.216) (width 0.5) (layer B.Cu) (net 7))
-  (segment (start 87.63 72.136) (end 88.9 70.866) (width 0.5) (layer B.Cu) (net 7))
+  (segment (start 87.63 72.136) (end 87.63 70.866) (width 0.5) (layer B.Cu) (net 7) (status 20))
   (segment (start 83.058 72.136) (end 87.63 72.136) (width 0.5) (layer B.Cu) (net 7))
   (segment (start 82.804 72.39) (end 83.058 72.136) (width 0.5) (layer B.Cu) (net 7))
@@
   (segment (start 56.388 69.596) (end 56.388 69.088) (width 0.5) (layer B.Cu) (net 10))
   (segment (start 55.372 70.612) (end 56.388 69.596) (width 0.5) (layer B.Cu) (net 10))
-  (segment (start 97.536 70.358) (end 96.52 70.358) (width 0.5) (layer B.Cu) (net 11))
-  (segment (start 86.36 68.58) (end 84.836 70.104) (width 0.5) (layer B.Cu) (net 11) (status 20))
+  (segment (start 96.012 70.866) (end 95.504 70.612) (width 0.5) (layer B.Cu) (net 11) (status 10))
+  (segment (start 86.36 68.58) (end 83.058 70.104) (width 0.5) (layer B.Cu) (net 11) (status 20))
   (segment (start 94.488 68.58) (end 86.36 68.58) (width 0.5) (layer B.Cu) (net 11))
-  (segment (start 96.52 70.358) (end 94.488 68.58) (width 0.5) (layer B.Cu) (net 11))
-  (segment (start 91.44 70.866) (end 92.964 70.866) (width 1) (layer B.Cu) (net 12))
+  (segment (start 95.504 70.612) (end 94.488 68.58) (width 0.5) (layer B.Cu) (net 11))
+  (segment (start 90.17 70.866) (end 92.964 70.866) (width 1) (layer B.Cu) (net 12) (status 10))
   (segment (start 95.25 73.152) (end 100.33 73.152) (width 1) (layer B.Cu) (net 12))
   (segment (start 92.964 70.866) (end 95.25 73.152) (width 1) (layer B.Cu) (net 12))
-  (segment (start 79.502 67.056) (end 100.33 67.056) (width 1) (layer B.Cu) (net 12))
-  (segment (start 99.314 81.788) (end 97.536 81.788) (width 1) (layer B.Cu) (net 12))
+  (segment (start 77.47 67.056) (end 100.33 67.056) (width 1) (layer B.Cu) (net 12))
+  (segment (start 99.314 81.788) (end 96.012 81.788) (width 1) (layer B.Cu) (net 12) (status 20))
   (segment (start 100.33 80.772) (end 99.314 81.788) (width 1) (layer B.Cu) (net 12))
   (segment (start 100.33 67.056) (end 100.33 73.152) (width 1) (layer B.Cu) (net 12))
   (segment (start 100.33 73.152) (end 100.33 80.772) (width 1) (layer B.Cu) (net 12))
-  (segment (start 79.502 67.056) (end 79.502 67.056) (width 0.5) (layer B.Cu) (net 12))
-  (segment (start 79.502 67.056) (end 70.866 67.056) (width 1) (layer B.Cu) (net 12))
+  (segment (start 77.47 67.056) (end 77.47 67.056) (width 0.5) (layer B.Cu) (net 12))
+  (segment (start 77.47 67.056) (end 70.866 67.056) (width 1) (layer B.Cu) (net 12))
   (segment (start 68.58 74.93) (end 59.944 74.93) (width 1) (layer B.Cu) (net 12))
   (segment (start 70.866 72.644) (end 70.866 67.056) (width 1) (layer B.Cu) (net 12))
@@
   (segment (start 67.564 78.486) (end 69.342 78.486) (width 1) (layer B.Cu) (net 12))
   (segment (start 69.342 78.486) (end 73.66 74.168) (width 1) (layer B.Cu) (net 12))
-  (segment (start 73.66 74.168) (end 79.248 74.168) (width 1) (layer B.Cu) (net 12))
-  (segment (start 79.248 74.168) (end 79.502 73.914) (width 0.5) (layer B.Cu) (net 12))
-  (segment (start 79.502 73.914) (end 79.502 67.056) (width 1) (layer B.Cu) (net 12))
+  (segment (start 73.66 74.168) (end 77.216 74.168) (width 1) (layer B.Cu) (net 12))
+  (segment (start 77.216 74.168) (end 77.47 73.914) (width 0.5) (layer B.Cu) (net 12))
+  (segment (start 77.47 73.914) (end 77.47 67.056) (width 1) (layer B.Cu) (net 12))
 )
