File: scheme/doorbell.kicad_pcb (KiCad board)
At the start: 2 copper layers, 50 x 25 mm, 15 parts

Commit message: next step
Parts:
- moved PIN_ARRAY_1 0.41 mm to (77.0, 89.4)
Routing:
- net (no net): track 150.0 -> 158.0 mm
- net GND: track 115.9 -> 117.9 mm
- net V+: track 101.1 -> 102.4 mm
Changed lines of the file:
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@@
-(kicad_pcb (version 3) (host pcbnew "(2013-jul-07)-stable")
+(kicad_pcb (version 3) (host pcbnew "(2013-07-07 BZR 4022)-stable")
   (general
     (links 22)
     (no_connects 0)
-    (area 51.873 65.27673 102.075001 92.075001)
+    (area 50.873 64.873 103.127001 92.127001)
     (thickness 1.6)
     (drawings 7)
-    (tracks 96)
+    (tracks 97)
     (zones 0)
     (modules 15)
@@
     (mod_text_size 1 1)
     (mod_text_width 0.15)
-    (pad_size 1.8 1.8)
+    (pad_size 3 3)
     (pad_drill 0.5)
     (pad_to_mask_clearance 0)
@@
     (visible_elements 7FFEE7CF)
     (pcbplotparams
-      (layerselection 3178497)
-      (usegerberextensions true)
+      (layerselection 1)
+      (usegerberextensions false)
       (excludeedgelayer true)
       (linewidth 0.150000)
@@
       (padsonsilk false)
       (subtractmaskfromsilk false)
-      (outputformat 1)
+      (outputformat 2)
       (mirror false)
-      (drillshape 1)
+      (drillshape 2)
       (scaleselection 1)
       (outputdirectory ""))
@@
     (fp_line (start -4.4902 3.5532) (end 5.5098 3.5532) (layer F.SilkS) (width 0.3))
     (fp_line (start 5.5098 3.5532) (end 5.5098 -3.4468) (layer F.SilkS) (width 0.3))
-    (pad 1 thru_hole circle (at -1.954 -0.396) (size 2 2) (drill 0.5)
+    (pad 1 thru_hole circle (at -1.954 -0.396) (size 3 3) (drill 0.5)
       (layers *.Cu *.Mask F.SilkS)
       (net 9 N-000005)
     )
-    (pad 2 thru_hole circle (at 0.586 2.144) (size 2 2) (drill 0.5)
-      (layers *.Cu *.Mask F.SilkS)
-      (net 1 GND)
-    )
-    (pad 3 thru_hole circle (at 3.126 -0.396) (size 2 2) (drill 0.5)
+    (pad 2 thru_hole circle (at 0.586 2.144) (size 3 3) (drill 0.5)
+      (layers *.Cu *.Mask F.SilkS)
+      (net 1 GND)
+    )
+    (pad 3 thru_hole circle (at 3.126 -0.396) (size 3 3) (drill 0.5)
       (layers *.Cu *.Mask F.SilkS)
       (net 2 N-000001)
@@
     (fp_line (start -5.08 -3.413) (end 4.953 -3.413) (layer F.SilkS) (width 0.3))
     (fp_line (start 5.08 3.54) (end -4.953 3.54) (layer F.SilkS) (width 0.3))
-    (pad 1 thru_hole circle (at -2.54 0 90) (size 2 2) (drill 0.5)
-      (layers *.Cu *.Mask F.SilkS)
-      (net 1 GND)
-    )
-    (pad 2 thru_hole circle (at 2.54 0 90) (size 2 2) (drill 0.5)
+    (pad 1 thru_hole oval (at -2.54 0 90) (size 2 3) (drill 0.5)
+      (layers *.Cu *.Mask F.SilkS)
+      (net 1 GND)
+    )
+    (pad 2 thru_hole oval (at 2.54 0 90) (size 2 3) (drill 0.5)
       (layers *.Cu *.Mask F.SilkS)
       (net 11 N-000009)
@@
     (fp_line (start -5.08 -3.413) (end 4.953 -3.413) (layer F.SilkS) (width 0.3))
     (fp_line (start 5.08 3.54) (end -4.953 3.54) (layer F.SilkS) (width 0.3))
-    (pad 1 thru_hole circle (at -2.54 0 270) (size 2 2) (drill 0.5)
+    (pad 1 thru_hole oval (at -2.54 0 270) (size 2 3) (drill 0.5)
       (layers *.Cu *.Mask F.SilkS)
       (net 12 V+)
     )
-    (pad 2 thru_hole circle (at 2.54 0 270) (size 2 2) (drill 0.5)
+    (pad 2 thru_hole oval (at 2.54 0 270) (size 2 3) (drill 0.5)
       (layers *.Cu *.Mask F.SilkS)
       (net 1 GND)
@@
   )
   (module PIN_ARRAY_1 (layer F.Cu)
-    (at 77 89)
+    (at 76.962 89.408)
     (descr "1 pin")
     (tags "CONN DEV")
@@
     (fp_line (start -1.27 1.27) (end -1.27 -1.27) (layer F.SilkS) (width 0.1524))
     (fp_line (start 1.27 -1.27) (end 1.27 1.27) (layer F.SilkS) (width 0.1524))
-    (pad 1 thru_hole rect (at 0 0) (size 1.524 1.524) (drill 1.016)
+    (pad 1 thru_hole rect (at 0 0) (size 1.524 1.524) (drill 0.5)
       (layers *.Cu *.Mask F.SilkS)
     )
@@
   (gr_line (start 102 66) (end 102 91) (angle 90) (layer Edge.Cuts) (width 0.15))
   (gr_line (start 52 66) (end 102 66) (angle 90) (layer Edge.Cuts) (width 0.15))
-  (segment (start 52 66) (end 52 91) (width 0.254) (layer B.Cu) (net 0))
-  (segment (start 102 66) (end 52 66) (width 0.254) (layer B.Cu) (net 0))
-  (segment (start 102 91) (end 102 66) (width 0.254) (layer B.Cu) (net 0))
-  (segment (start 52 91) (end 102 91) (width 0.254) (layer B.Cu) (net 0))
+  (segment (start 51 65) (end 51 92) (width 0.254) (layer B.Cu) (net 0))
+  (segment (start 103 65) (end 51 65) (width 0.254) (layer B.Cu) (net 0))
+  (segment (start 103 92) (end 103 65) (width 0.254) (layer B.Cu) (net 0))
+  (segment (start 51 92) (end 103 92) (width 0.254) (layer B.Cu) (net 0))
+  (segment (start 96.012 75.946) (end 96.012 77.978) (width 1) (layer B.Cu) (net 1) (status 400000))
+  (segment (start 96.012 77.978) (end 92.456 77.978) (width 1) (layer B.Cu) (net 1))
+  (segment (start 96.012 86.868) (end 93.726 86.868) (width 1) (layer B.Cu) (net 1))
+  (segment (start 93.218 86.36) (end 90.424 86.36) (width 1) (layer B.Cu) (net 1))
+  (segment (start 93.726 86.868) (end 93.218 86.36) (width 1) (layer B.Cu) (net 1))
   (segment (start 59.944 86.106) (end 60.198 86.106) (width 0.5) (layer B.Cu) (net 1))
   (segment (start 94.996 89.408) (end 96.012 86.868) (width 1) (layer B.Cu) (net 1) (status 20))
@@
   (segment (start 60.198 86.106) (end 62.738 88.646) (width 1) (layer B.Cu) (net 1))
   (segment (start 77.04 81.646) (end 77.836 81.646) (width 1) (layer B.Cu) (net 1))
+  (segment (start 77.836 81.646) (end 79.756 83.566) (width 1) (layer B.Cu) (net 1))
+  (segment (start 79.756 83.566) (end 84.074 84.074) (width 1) (layer B.Cu) (net 1))
+  (segment (start 84.074 84.074) (end 86.868 86.36) (width 1) (layer B.Cu) (net 1))
   (segment (start 86.868 86.36) (end 90.424 86.36) (width 1) (layer B.Cu) (net 1))
-  (segment (start 84.074 84.074) (end 86.868 86.36) (width 1) (layer B.Cu) (net 1))
-  (segment (start 79.756 83.566) (end 84.074 84.074) (width 1) (layer B.Cu) (net 1))
-  (segment (start 77.836 81.646) (end 79.756 83.566) (width 1) (layer B.Cu) (net 1))
-  (segment (start 96.012 86.868) (end 93.218 86.868) (width 1) (layer B.Cu) (net 1) (status 10))
-  (segment (start 91.186 86.36) (end 90.424 86.36) (width 0.5) (layer B.Cu) (net 1) (status 30))
-  (segment (start 93.218 86.868) (end 91.186 86.36) (width 1) (layer B.Cu) (net 1) (status 20))
   (segment (start 85.598 79.756) (end 89.154 79.756) (width 1) (layer B.Cu) (net 1))
-  (segment (start 90.932 77.978) (end 93.218 77.978) (width 1) (layer B.Cu) (net 1))
+  (segment (start 90.932 77.978) (end 92.456 77.978) (width 1) (layer B.Cu) (net 1))
+  (segment (start 92.456 77.978) (end 92.71 77.978) (width 1) (layer B.Cu) (net 1))
   (segment (start 89.154 79.756) (end 90.932 77.978) (width 1) (layer B.Cu) (net 1))
   (segment (start 58.928 69.088) (end 58.928 70.612) (width 1) (layer B.Cu) (net 1))
@@
   (segment (start 57.658 71.882) (end 57.658 77.47) (width 1) (layer B.Cu) (net 1))
   (segment (start 58.928 70.612) (end 57.658 71.882) (width 1) (layer B.Cu) (net 1))
-  (segment (start 96.012 86.868) (end 93.218 83.312) (width 1) (layer B.Cu) (net 1) (status 400010))
-  (segment (start 93.218 83.312) (end 93.218 77.978) (width 1) (layer B.Cu) (net 1))
-  (segment (start 95.504 75.946) (end 96.012 75.946) (width 0.5) (layer B.Cu) (net 1) (status 30))
-  (segment (start 93.218 77.978) (end 95.504 75.946) (width 1) (layer B.Cu) (net 1) (status 20))
+  (segment (start 96.012 86.868) (end 92.71 83.312) (width 1) (layer B.Cu) (net 1) (status 400010))
+  (segment (start 92.71 83.312) (end 92.71 77.978) (width 1) (layer B.Cu) (net 1))
   (segment (start 58.928 69.088) (end 64.008 69.088) (width 1) (layer B.Cu) (net 1) (status 20))
   (segment (start 90.424 82.296) (end 82.804 82.296) (width 0.5) (layer B.Cu) (net 2))
@@
   (segment (start 95.504 70.612) (end 94.488 68.58) (width 0.5) (layer B.Cu) (net 11))
   (segment (start 90.17 70.866) (end 92.964 70.866) (width 1) (layer B.Cu) (net 12) (status 10))
-  (segment (start 95.25 73.152) (end 100.33 73.152) (width 1) (layer B.Cu) (net 12))
-  (segment (start 92.964 70.866) (end 95.25 73.152) (width 1) (layer B.Cu) (net 12))
+  (segment (start 92.964 73.152) (end 100.33 73.152) (width 1) (layer B.Cu) (net 12))
+  (segment (start 92.964 70.866) (end 92.964 73.152) (width 1) (layer B.Cu) (net 12))
   (segment (start 77.47 67.056) (end 100.33 67.056) (width 1) (layer B.Cu) (net 12))
   (segment (start 99.314 81.788) (end 96.012 81.788) (width 1) (layer B.Cu) (net 12) (status 20))
