File: scheme/doorbell.kicad_pcb (KiCad board)
At the start: 2 copper layers, 50 x 25 mm, 15 parts

Commit message: small changes
Parts:
- removed PIN_ARRAY_1: Val**, PIN_ARRAY_1
Connections:
- R1 pad 2: N-000001 (its old number) -> N-000009
- R2 pad 2: GND -> N-000009
- R2 pad 3: N-000001 (its old number) -> GND
Routing:
- net N-000009: track 0.00 -> 13.7 mm
- net N-000001 (its old number): track 12.2 -> 0.00 mm
- net GND: track 115.9 -> 107.1 mm

Commit message: small changes
Parts:
- added XS3: питание радиомодуля, SIL-2, F.Cu at (68.8, 68.8)
- R1: value 5,1к -> 3,6к
- moved VD2 2.81 mm to (62.5, 68.8)
- moved VD1 1.80 mm to (55.9, 68.8)
- moved XS2 1.02 mm to (75.2, 69.6)
Routing:
- net GND: track 107.1 -> 117.2 mm
- net N-000003: track 4.08 -> 7.87 mm
- net V+: track 101.1 -> 103.8 mm
