File: scheme/doorbell.sch (KiCad schematic (older format))
At the start: 0 parts

Commit message: next step
Parts:
- added DD1: ATTINY45, symbol GIC_ATTINY13
- added R1, R2: RES, symbol RES
- added R3: RES_VAR, symbol RES_VAR
- added VT1: КТ315, symbol TR_NPN_BCE
- added XS1: Питание, symbol CONN_02_F
- added XS2: Динамик, symbol CONN_02_F
- added XS3: Кнопки, symbol CONN_02_F
- added XS4: Геркон, symbol CONN_02_F
Connections:
- new net: R1.1, R3.2, R3.3
- new net: DD1.6 (PB1), R1.2
- new net: R3.1, VT1.1 (B)
- new net: VT1.2 (C), XS2.2
- new net: DD1.5 (PB0), XS3.1
- new net: DD1.7 (PB2), R2.1, XS3.2
- new net: R2.2, XS4.1
- new net GND: DD1.4 (GND), VT1.3 (E), XS1.2, XS4.2
- new net V+: DD1.1 (RES), DD1.8 (VCC), XS1.1, XS2.1
- no-connect marks 0 -> 2

Commit message: next step
Parts:
- removed XS2: Динамик, symbol CONN_02_F
- removed XS4: Геркон, symbol CONN_02_F
- added SF1: SF, ~, symbol SF
- added SP1: SPEAKER, ~, symbol SPEAKER
Connections:
- net GND: now also SF1.1
- net V+: now also SP1.1
- net at VT1.2 (C): now also SP1.2
- net at R2.2: now also SF1.2
Changed lines of the file:
@@
 LIBS:valves
 LIBS:gost
+LIBS:mixture
 LIBS:doorbell-cache
 EELAYER 27 0
@@
 $EndComp
 $Comp
-L CONN_02_F XS2
-U 1 1 53144DBF
-P 6850 3900
-F 0 "XS2" H 7100 4000 60  0000 C CNN
-F 1 "Динамик" H 7200 3675 60  0000 C CNN
-F 2 "" H 6850 3900 60  0000 C CNN
-F 3 "" H 6850 3900 60  0000 C CNN
-	1    6850 3900
-	1    0    0    -1
-$EndComp
-$Comp
 L CONN_02_F XS3
 U 1 1 53144DCE
@@
 L POWER_GND #04
 U 1 1 53145822
-P 6325 1700
-F 0 "#04" V 6275 1650 60  0001 C CNN
-F 1 "POWER_GND" V 6375 1650 60  0001 C CNN
-F 2 "" H 6325 1700 60  0000 C CNN
-F 3 "" H 6325 1700 60  0000 C CNN
-	1    6325 1700
+P 7025 1600
+F 0 "#04" V 6975 1550 60  0001 C CNN
+F 1 "POWER_GND" V 7075 1550 60  0001 C CNN
+F 2 "" H 7025 1600 60  0000 C CNN
+F 3 "" H 7025 1600 60  0000 C CNN
+	1    7025 1600
 	1    0    0    -1
 $EndComp
@@
 $EndComp
 Wire Wire Line
-	3725 2775 4325 2775
+	3725 2775 3975 2775
+Wire Wire Line
+	3975 2775 4275 2775
+Wire Wire Line
+	4275 2775 4325 2775
 Wire Wire Line
 	5325 2775 5450 2775
@@
 	6325 2575 6325 2275
 Wire Wire Line
-	5325 2575 6325 2575
+	5325 2575 5700 2575
+Wire Wire Line
+	5700 2575 6325 2575
 Wire Wire Line
 	6850 4850 6850 4700
 Wire Wire Line
-	6325 1700 6325 1300
+	7025 1600 7025 1200
 Wire Wire Line
 	5700 2075 5700 2575
@@
 $EndComp
 Wire Wire Line
-	3725 2175 4325 2175
+	3725 2175 3875 2175
+Wire Wire Line
+	3875 2175 4100 2175
+Wire Wire Line
+	4100 2175 4325 2175
 Wire Wire Line
 	3875 2175 3875 2000
@@
 Wire Wire Line
 	6000 3550 6000 3450
-$Comp
-L CONN_02_F XS4
-U 1 1 53144E85
-P 6325 1200
-F 0 "XS4" H 6575 1300 60  0000 C CNN
-F 1 "Геркон" H 6675 975 60  0000 C CNN
-F 2 "" H 6325 1200 60  0000 C CNN
-F 3 "" H 6325 1200 60  0000 C CNN
-	1    6325 1200
-	1    0    0    -1
-$EndComp
-Wire Wire Line
-	6325 1200 5700 1200
+Wire Wire Line
+	6425 1200 5700 1200
 Wire Wire Line
 	5700 1200 5700 1275
@@
 L POWER_V+ #07
 U 1 1 53145AD3
-P 6850 3775
-F 0 "#07" V 6650 3525 60  0001 C CNN
-F 1 "POWER_V+" H 7000 3675 60  0001 C CNN
-F 2 "" H 6850 3775 60  0000 C CNN
-F 3 "" H 6850 3775 60  0000 C CNN
-	1    6850 3775
+P 6850 3475
+F 0 "#07" V 6650 3225 60  0001 C CNN
+F 1 "POWER_V+" H 7000 3375 60  0001 C CNN
+F 2 "" H 6850 3475 60  0000 C CNN
+F 3 "" H 6850 3475 60  0000 C CNN
+	1    6850 3475
 	0    -1   -1   0
 $EndComp
@@
 	4100 2075 4100 2175
 Connection ~ 4100 2175
-Wire Wire Line
-	6850 4000 6850 4100
-Wire Wire Line
-	6850 3900 6850 3775
+$Comp
+L SPEAKER SP1
+U 1 1 531471A4
+P 7100 3900
+F 0 "SP1" H 7075 4100 70  0000 C CNN
+F 1 "SPEAKER" H 7000 3650 70  0001 C CNN
+F 2 "~" H 7100 3900 60  0000 C CNN
+F 3 "~" H 7100 3900 60  0000 C CNN
+	1    7100 3900
+	1    0    0    -1
+$EndComp
+Wire Wire Line
+	6850 4100 6850 4000
+Wire Wire Line
+	6850 3800 6850 3475
+$Comp
+L SF SF1
+U 1 1 5314886A
+P 6725 1200
+F 0 "SF1" H 6725 1450 47  0000 C CNN
+F 1 "SF" H 5125 2100 60  0001 C CNN
+F 2 "~" H 6725 1200 60  0000 C CNN
+F 3 "~" H 6725 1200 60  0000 C CNN
+	1    6725 1200
+	1    0    0    -1
+$EndComp
 $EndSCHEMATC

Commit message: next step
Changed lines of the file:
@@
 $EndComp
 Wire Wire Line
-	3725 2775 3975 2775
-Wire Wire Line
-	3975 2775 4275 2775
-Wire Wire Line
-	4275 2775 4325 2775
+	3725 2775 4325 2775
 Wire Wire Line
 	5325 2775 5450 2775
@@
 	6325 2575 6325 2275
 Wire Wire Line
-	5325 2575 5700 2575
-Wire Wire Line
-	5700 2575 6325 2575
+	5325 2575 6325 2575
 Wire Wire Line
 	6850 4850 6850 4700
@@
 $EndComp
 Wire Wire Line
-	3725 2175 3875 2175
-Wire Wire Line
-	3875 2175 4100 2175
-Wire Wire Line
-	4100 2175 4325 2175
+	3725 2175 4325 2175
 Wire Wire Line
 	3875 2175 3875 2000
@@
 P 6725 1200
 F 0 "SF1" H 6725 1450 47  0000 C CNN
-F 1 "SF" H 5125 2100 60  0001 C CNN
+F 1 "SF" H 4800 -925 60  0001 C CNN
 F 2 "~" H 6725 1200 60  0000 C CNN
 F 3 "~" H 6725 1200 60  0000 C CNN

Commit message: next step
Parts:
- removed R2: RES, symbol RES
- removed XS3: Кнопки, symbol CONN_02_F
- added R3, R4: 100, ~, symbol RES
- added SA1: SA, ~, symbol SA
- added VD1, VD2: LED, ~, symbol LED
- added XS2: пуск, symbol CONN_01_F
- R1: value RES -> 5,1к
- R2: renamed from R3; value RES_VAR -> 1к
Connections:
- net GND: now also R2.2, VD1.1, VD2.1
- net V+: now also R4.2
- net at R1.2: now also R2.3; no longer DD1.6 (PB1)
- net at VT1.1 (B): now also R1.1; no longer R2.1
- net at DD1.2 (PB3): now also R3.2
- net at DD1.5 (PB0): now also XS2.1
- net at DD1.7 (PB2): now also SA1.2
- net at SF1.2: now also SA1.1
- new net: DD1.6 (PB1), R2.1
- new net: R4.1, VD2.2
- new net: R3.1, VD1.2
- no-connect marks 2 -> 1
Other:
- moved on the sheet: R1, R2, XS1
Changed lines of the file:
@@
 EESchema Schematic File Version 2
 LIBS:power
-LIBS:device
 LIBS:transistors
 LIBS:conn
@@
 Sheet 1 1
 Title ""
-Date "3 mar 2014"
+Date "4 mar 2014"
 Rev ""
 Comp ""
@@
 L RES R1
 U 1 1 53144C3F
-P 6000 3450
-F 0 "R1" H 6250 3575 60  0000 C CNN
-F 1 "RES" H 6275 3300 60  0000 C CNN
-F 2 "" H 6000 3450 60  0000 C CNN
-F 3 "" H 6000 3450 60  0000 C CNN
-	1    6000 3450
+P 6000 4400
+F 0 "R1" V 6550 4575 60  0000 C CNN
+F 1 "5,1к" V 6400 4175 60  0000 C CNN
+F 2 "" H 6000 4400 60  0000 C CNN
+F 3 "" H 6000 4400 60  0000 C CNN
+	1    6000 4400
 	0    -1   -1   0
 $EndComp
@@
 L CONN_02_F XS1
 U 1 1 53144DB0
-P 3725 2175
-F 0 "XS1" H 3975 2275 60  0000 C CNN
-F 1 "Питание" H 4050 1950 60  0000 C CNN
-F 2 "" H 3725 2175 60  0000 C CNN
-F 3 "" H 3725 2175 60  0000 C CNN
-	1    3725 2175
+P 3350 2275
+F 0 "XS1" H 3600 2375 60  0000 C CNN
+F 1 "Питание" H 3675 2050 60  0000 C CNN
+F 2 "" H 3350 2275 60  0000 C CNN
+F 3 "" H 3350 2275 60  0000 C CNN
+	1    3350 2275
 	-1   0    0    -1
-$EndComp
-$Comp
-L CONN_02_F XS3
-U 1 1 53144DCE
-P 6325 2175
-F 0 "XS3" H 6575 2275 60  0000 C CNN
-F 1 "Кнопки" H 6675 1950 60  0000 C CNN
-F 2 "" H 6325 2175 60  0000 C CNN
-F 3 "" H 6325 2175 60  0000 C CNN
-	1    6325 2175
-	1    0    0    -1
 $EndComp
 $Comp
@@
 $EndComp
 $Comp
-L RES_VAR R3
-U 1 1 53144F7E
-P 6000 4350
-F 0 "R3" H 6250 4475 60  0000 C CNN
-F 1 "RES_VAR" H 6425 4225 60  0000 C CNN
-F 2 "" H 6000 4350 60  0000 C CNN
-F 3 "" H 6000 4350 60  0000 C CNN
-	1    6000 4350
-	0    -1   -1   0
-$EndComp
-$Comp
-L RES R2
-U 1 1 53145720
-P 5700 2075
-F 0 "R2" H 5950 2200 60  0000 C CNN
-F 1 "RES" H 5975 1925 60  0000 C CNN
-F 2 "" H 5700 2075 60  0000 C CNN
-F 3 "" H 5700 2075 60  0000 C CNN
-	1    5700 2075
-	0    -1   -1   0
-$EndComp
-$Comp
 L POWER_GND #04
 U 1 1 53145822
@@
 $EndComp
 NoConn ~ 4325 2575
-NoConn ~ 4325 2375
 $Comp
 L POWER_V+ #05
@@
 	0    -1   -1   0
 $EndComp
-Wire Wire Line
-	3725 2775 4325 2775
-Wire Wire Line
-	5325 2775 5450 2775
-Wire Wire Line
-	5325 2175 6325 2175
-Wire Wire Line
-	6325 2575 6325 2275
-Wire Wire Line
-	5325 2575 6325 2575
-Wire Wire Line
-	6850 4850 6850 4700
-Wire Wire Line
-	7025 1600 7025 1200
-Wire Wire Line
-	5700 2075 5700 2575
-Connection ~ 5700 2575
 $Comp
 L PWR_FLAG #FLG06
 U 1 1 531473BB
-P 3975 2675
-F 0 "#FLG06" H 3975 2770 30  0001 C CNN
-F 1 "PWR_FLAG" H 3975 2855 30  0000 C CNN
-F 2 "" H 3975 2675 60  0000 C CNN
-F 3 "" H 3975 2675 60  0000 C CNN
-	1    3975 2675
-	1    0    0    -1
-$EndComp
-Wire Wire Line
-	3725 2175 4325 2175
-Wire Wire Line
-	3875 2175 3875 2000
-Wire Wire Line
-	5800 3550 6000 3550
-Wire Wire Line
-	6000 3550 6000 3450
-Wire Wire Line
-	6425 1200 5700 1200
-Wire Wire Line
-	5700 1200 5700 1275
-Connection ~ 3875 2175
-Wire Wire Line
-	3725 2775 3725 2275
-Connection ~ 4275 2775
-Wire Wire Line
-	5325 2375 6000 2375
-Wire Wire Line
-	6000 2375 6000 2650
-Wire Wire Line
-	6400 4400 6000 4400
-Wire Wire Line
-	6000 4400 6000 4350
+P 3150 2775
+F 0 "#FLG06" H 3150 2870 30  0001 C CNN
+F 1 "PWR_FLAG" H 3150 2955 30  0000 C CNN
+F 2 "" H 3150 2775 60  0000 C CNN
+F 3 "" H 3150 2775 60  0000 C CNN
+	1    3150 2775
+	1    0    0    -1
+$EndComp
 $Comp
 L POWER_V+ #07
@@
 	1    0    0    -1
 $EndComp
-Wire Wire Line
-	3975 2675 3975 2775
-Connection ~ 3975 2775
-Wire Wire Line
-	4100 2075 4100 2175
-Connection ~ 4100 2175
 $Comp
 L SPEAKER SP1
@@
 	1    0    0    -1
 $EndComp
-Wire Wire Line
-	6850 4100 6850 4000
-Wire Wire Line
-	6850 3800 6850 3475
 $Comp
 L SF SF1
@@
 	1    0    0    -1
 $EndComp
+$Comp
+L RES R4
+U 1 1 5315BF3A
+P 3475 3875
+F 0 "R4" V 4075 4050 60  0000 C CNN
+F 1 "100" V 3850 3675 60  0000 C CNN
+F 2 "~" H 3475 3875 60  0000 C CNN
+F 3 "~" H 3475 3875 60  0000 C CNN
+	1    3475 3875
+	0    -1   -1   0
+$EndComp
+$Comp
+L LED VD2
+U 1 1 5315D934
+P 3475 4275
+F 0 "VD2" V 3600 4500 60  0000 C CNN
+F 1 "LED" H 3525 4075 60  0001 C CNN
+F 2 "~" H 3475 4275 60  0000 C CNN
+F 3 "~" H 3475 4275 60  0000 C CNN
+	1    3475 4275
+	0    -1   -1   0
+$EndComp
+$Comp
+L POWER_GND #09
+U 1 1 5315D992
+P 3475 4650
+F 0 "#09" V 3425 4600 60  0001 C CNN
+F 1 "POWER_GND" V 3525 4600 60  0001 C CNN
+F 2 "" H 3475 4650 60  0000 C CNN
+F 3 "" H 3475 4650 60  0000 C CNN
+	1    3475 4650
+	1    0    0    -1
+$EndComp
+$Comp
+L RES_VAR R2
+U 1 1 53144F7E
+P 6000 2650
+F 0 "R2" V 6275 2800 60  0000 C CNN
+F 1 "1к" V 6400 2500 60  0000 C CNN
+F 2 "" H 6000 2650 60  0000 C CNN
+F 3 "" H 6000 2650 60  0000 C CNN
+	1    6000 2650
+	0    -1   1    0
+$EndComp
+$Comp
+L POWER_GND #010
+U 1 1 5315D9B8
+P 5500 3450
+F 0 "#010" V 5450 3400 60  0001 C CNN
+F 1 "POWER_GND" V 5550 3400 60  0001 C CNN
+F 2 "" H 5500 3450 60  0000 C CNN
+F 3 "" H 5500 3450 60  0000 C CNN
+	1    5500 3450
+	1    0    0    -1
+$EndComp
+$Comp
+L RES R3
+U 1 1 5315DB42
+P 4025 3875
+F 0 "R3" V 4650 4025 60  0000 C CNN
+F 1 "100" V 4400 3675 60  0000 C CNN
+F 2 "~" H 4025 3875 60  0000 C CNN
+F 3 "~" H 4025 3875 60  0000 C CNN
+	1    4025 3875
+	0    -1   -1   0
+$EndComp
+$Comp
+L LED VD1
+U 1 1 5315DB48
+P 4025 4275
+F 0 "VD1" V 4150 4500 60  0000 C CNN
+F 1 "LED" H 4075 4075 60  0001 C CNN
+F 2 "~" H 4025 4275 60  0000 C CNN
+F 3 "~" H 4025 4275 60  0000 C CNN
+	1    4025 4275
+	0    -1   -1   0
+$EndComp
+$Comp
+L POWER_GND #011
+U 1 1 5315DB4E
+P 4025 4650
+F 0 "#011" V 3975 4600 60  0001 C CNN
+F 1 "POWER_GND" V 4075 4600 60  0001 C CNN
+F 2 "" H 4025 4650 60  0000 C CNN
+F 3 "" H 4025 4650 60  0000 C CNN
+	1    4025 4650
+	1    0    0    -1
+$EndComp
+Wire Wire Line
+	3150 2775 4325 2775
+Wire Wire Line
+	5325 2775 5450 2775
+Wire Wire Line
+	5325 2175 6325 2175
+Wire Wire Line
+	6850 4850 6850 4700
+Wire Wire Line
+	7025 1600 7025 1200
+Wire Wire Line
+	3350 2175 4325 2175
+Wire Wire Line
+	3875 2175 3875 2000
+Wire Wire Line
+	6000 3600 6000 3450
+Wire Wire Line
+	6425 1200 5700 1200
+Connection ~ 3875 2175
+Connection ~ 4275 2775
+Wire Wire Line
+	5325 2375 6000 2375
+Wire Wire Line
+	6000 2375 6000 2650
+Wire Wire Line
+	6400 4400 6000 4400
+Wire Wire Line
+	4100 2075 4100 2175
+Connection ~ 4100 2175
+Wire Wire Line
+	6850 4100 6850 4000
+Wire Wire Line
+	6850 3800 6850 3475
+Wire Wire Line
+	4325 2375 4025 2375
+Wire Wire Line
+	4025 2375 4025 3075
+Wire Wire Line
+	3475 3875 3475 4025
+Wire Wire Line
+	3475 4525 3475 4650
+Wire Wire Line
+	4025 4650 4025 4525
+Wire Wire Line
+	4025 4025 4025 3875
+Wire Wire Line
+	3350 2775 3350 2375
+Wire Wire Line
+	3475 3075 3475 2175
+Wire Wire Line
+	3350 2175 3350 2275
+Connection ~ 3475 2175
+Connection ~ 3350 2775
+Wire Wire Line
+	5800 3450 5500 3450
+$Comp
+L SA SA1
+U 1 1 5315E094
+P 5700 1575
+F 0 "SA1" V 5700 1775 60  0000 C CNN
+F 1 "SA" H 5700 1475 60  0001 C CNN
+F 2 "~" H 5700 1575 60  0000 C CNN
+F 3 "~" H 5700 1575 60  0000 C CNN
+	1    5700 1575
+	0    -1   -1   0
+$EndComp
+Wire Wire Line
+	5700 1775 5700 2575
+Wire Wire Line
+	5700 2575 5325 2575
+Wire Wire Line
+	5700 1200 5700 1375
+$Comp
+L CONN_01_F XS2
+U 1 1 5315E124
+P 6325 2175
+F 0 "XS2" H 6575 2275 60  0000 C CNN
+F 1 "пуск" H 6675 2075 60  0000 C CNN
+F 2 "" H 6325 2175 60  0000 C CNN
+F 3 "" H 6325 2175 60  0000 C CNN
+	1    6325 2175
+	1    0    0    -1
+$EndComp

Commit message: next step
Parts:
- added R5: 3,6к, ~, symbol RES
- VD1: value LED -> красный
- VD2: value LED -> зеленый
Connections:
- net GND: now also R5.1
- net at DD1.5 (PB0), XS2.1: now also R5.2
Other:
- moved on the sheet: SP1, VT1, XS2
Changed lines of the file:
@@
 L TR_NPN_BCE VT1
 U 1 1 53144C4E
-P 6400 4400
-F 0 "VT1" H 6800 4600 60  0000 R CNN
-F 1 "КТ315" H 6800 4200 60  0000 R CNN
-F 2 "" H 6400 4400 60  0000 C CNN
-F 3 "" H 6400 4400 60  0000 C CNN
-	1    6400 4400
+P 6900 4400
+F 0 "VT1" H 7300 4600 60  0000 R CNN
+F 1 "КТ315" H 7300 4200 60  0000 R CNN
+F 2 "" H 6900 4400 60  0000 C CNN
+F 3 "" H 6900 4400 60  0000 C CNN
+	1    6900 4400
 	1    0    0    -1
 $EndComp
@@
 L POWER_GND #03
 U 1 1 53144F64
-P 6850 4850
-F 0 "#03" V 6800 4800 60  0001 C CNN
-F 1 "POWER_GND" V 6900 4800 60  0001 C CNN
-F 2 "" H 6850 4850 60  0000 C CNN
-F 3 "" H 6850 4850 60  0000 C CNN
-	1    6850 4850
+P 7350 4850
+F 0 "#03" V 7300 4800 60  0001 C CNN
+F 1 "POWER_GND" V 7400 4800 60  0001 C CNN
+F 2 "" H 7350 4850 60  0000 C CNN
+F 3 "" H 7350 4850 60  0000 C CNN
+	1    7350 4850
 	1    0    0    -1
 $EndComp
@@
 P 3150 2775
 F 0 "#FLG06" H 3150 2870 30  0001 C CNN
-F 1 "PWR_FLAG" H 3150 2955 30  0000 C CNN
+F 1 "PWR_FLAG" H 3150 2925 30  0000 C CNN
 F 2 "" H 3150 2775 60  0000 C CNN
 F 3 "" H 3150 2775 60  0000 C CNN
@@
 L POWER_V+ #07
 U 1 1 53145AD3
-P 6850 3475
-F 0 "#07" V 6650 3225 60  0001 C CNN
-F 1 "POWER_V+" H 7000 3375 60  0001 C CNN
-F 2 "" H 6850 3475 60  0000 C CNN
-F 3 "" H 6850 3475 60  0000 C CNN
-	1    6850 3475
+P 7350 3475
+F 0 "#07" V 7150 3225 60  0001 C CNN
+F 1 "POWER_V+" H 7500 3375 60  0001 C CNN
+F 2 "" H 7350 3475 60  0000 C CNN
+F 3 "" H 7350 3475 60  0000 C CNN
+	1    7350 3475
 	0    -1   -1   0
 $EndComp
@@
 P 4100 2075
 F 0 "#FLG08" H 4100 2170 30  0001 C CNN
-F 1 "PWR_FLAG" H 4100 2255 30  0000 C CNN
+F 1 "PWR_FLAG" H 4100 2225 30  0000 C CNN
 F 2 "" H 4100 2075 60  0000 C CNN
 F 3 "" H 4100 2075 60  0000 C CNN
@@
 L SPEAKER SP1
 U 1 1 531471A4
-P 7100 3900
-F 0 "SP1" H 7075 4100 70  0000 C CNN
-F 1 "SPEAKER" H 7000 3650 70  0001 C CNN
-F 2 "~" H 7100 3900 60  0000 C CNN
-F 3 "~" H 7100 3900 60  0000 C CNN
-	1    7100 3900
+P 7600 3900
+F 0 "SP1" H 7575 4100 70  0000 C CNN
+F 1 "SPEAKER" H 7500 3650 70  0001 C CNN
+F 2 "~" H 7600 3900 60  0000 C CNN
+F 3 "~" H 7600 3900 60  0000 C CNN
+	1    7600 3900
 	1    0    0    -1
 $EndComp
@@
 U 1 1 5315D934
 P 3475 4275
-F 0 "VD2" V 3600 4500 60  0000 C CNN
-F 1 "LED" H 3525 4075 60  0001 C CNN
+F 0 "VD2" V 3600 4450 60  0000 C CNN
+F 1 "зеленый" V 3475 4600 60  0000 C CNN
 F 2 "~" H 3475 4275 60  0000 C CNN
 F 3 "~" H 3475 4275 60  0000 C CNN
@@
 U 1 1 5315DB48
 P 4025 4275
-F 0 "VD1" V 4150 4500 60  0000 C CNN
-F 1 "LED" H 4075 4075 60  0001 C CNN
+F 0 "VD1" V 4175 4400 60  0000 C CNN
+F 1 "красный" V 4050 3900 60  0000 C CNN
 F 2 "~" H 4025 4275 60  0000 C CNN
 F 3 "~" H 4025 4275 60  0000 C CNN
@@
 	5325 2775 5450 2775
 Wire Wire Line
-	5325 2175 6325 2175
-Wire Wire Line
-	6850 4850 6850 4700
+	5325 2175 6925 2175
+Wire Wire Line
+	7350 4850 7350 4700
 Wire Wire Line
 	7025 1600 7025 1200
@@
 	6000 2375 6000 2650
 Wire Wire Line
-	6400 4400 6000 4400
+	6900 4400 6000 4400
 Wire Wire Line
 	4100 2075 4100 2175
 Connection ~ 4100 2175
 Wire Wire Line
-	6850 4100 6850 4000
-Wire Wire Line
-	6850 3800 6850 3475
+	7350 4100 7350 4000
+Wire Wire Line
+	7350 3800 7350 3475
 Wire Wire Line
 	4325 2375 4025 2375
@@
 L CONN_01_F XS2
 U 1 1 5315E124
-P 6325 2175
-F 0 "XS2" H 6575 2275 60  0000 C CNN
-F 1 "пуск" H 6675 2075 60  0000 C CNN
-F 2 "" H 6325 2175 60  0000 C CNN
-F 3 "" H 6325 2175 60  0000 C CNN
-	1    6325 2175
-	1    0    0    -1
-$EndComp
+P 6925 2175
+F 0 "XS2" H 7175 2275 60  0000 C CNN
+F 1 "пуск" H 7275 2075 60  0000 C CNN
+F 2 "" H 6925 2175 60  0000 C CNN
+F 3 "" H 6925 2175 60  0000 C CNN
+	1    6925 2175
+	1    0    0    -1
+$EndComp
+$Comp
+L RES R5
+U 1 1 5315E669
+P 6550 2975
+F 0 "R5" V 7125 3150 60  0000 C CNN
+F 1 "3,6к" V 6800 2725 60  0000 C CNN
+F 2 "~" H 6550 2975 60  0000 C CNN
+F 3 "~" H 6550 2975 60  0000 C CNN
+	1    6550 2975
+	0    -1   -1   0
+$EndComp
+Connection ~ 6550 2175
+$Comp
+L POWER_GND #?
+U 1 1 5315E6C5
+P 6550 3075
+F 0 "#?" V 6500 3025 60  0001 C CNN
+F 1 "POWER_GND" V 6600 3025 60  0001 C CNN
+F 2 "" H 6550 3075 60  0000 C CNN
+F 3 "" H 6550 3075 60  0000 C CNN
+	1    6550 3075
+	1    0    0    -1
+$EndComp
+Wire Wire Line
+	6550 3075 6550 2975
 $EndSCHEMATC

Commit message: small changes
Connections:
- net GND: now also R2.3; no longer R2.2
- net at R1.2: now also R2.2; no longer R2.3
Other:
- moved on the sheet: R1
Changed lines of the file:
@@
 Sheet 1 1
 Title ""
-Date "4 mar 2014"
+Date "8 mar 2014"
 Rev ""
 Comp ""
@@
 L RES R1
 U 1 1 53144C3F
-P 6000 4400
-F 0 "R1" V 6550 4575 60  0000 C CNN
-F 1 "5,1к" V 6400 4175 60  0000 C CNN
-F 2 "" H 6000 4400 60  0000 C CNN
-F 3 "" H 6000 4400 60  0000 C CNN
-	1    6000 4400
+P 5800 4400
+F 0 "R1" V 6350 4575 60  0000 C CNN
+F 1 "5,1к" V 6200 4175 60  0000 C CNN
+F 2 "" H 5800 4400 60  0000 C CNN
+F 3 "" H 5800 4400 60  0000 C CNN
+	1    5800 4400
 	0    -1   -1   0
 $EndComp
@@
 $EndComp
 $Comp
-L POWER_GND #010
-U 1 1 5315D9B8
-P 5500 3450
-F 0 "#010" V 5450 3400 60  0001 C CNN
-F 1 "POWER_GND" V 5550 3400 60  0001 C CNN
-F 2 "" H 5500 3450 60  0000 C CNN
-F 3 "" H 5500 3450 60  0000 C CNN
-	1    5500 3450
-	1    0    0    -1
-$EndComp
-$Comp
 L RES R3
 U 1 1 5315DB42
@@
 $EndComp
 $Comp
-L POWER_GND #011
+L POWER_GND #010
 U 1 1 5315DB4E
 P 4025 4650
-F 0 "#011" V 3975 4600 60  0001 C CNN
+F 0 "#010" V 3975 4600 60  0001 C CNN
 F 1 "POWER_GND" V 4075 4600 60  0001 C CNN
 F 2 "" H 4025 4650 60  0000 C CNN
@@
 $EndComp
 Wire Wire Line
-	3150 2775 4325 2775
+	3150 2775 3350 2775
+Wire Wire Line
+	3350 2775 4275 2775
+Wire Wire Line
+	4275 2775 4325 2775
 Wire Wire Line
 	5325 2775 5450 2775
 Wire Wire Line
-	5325 2175 6925 2175
+	5325 2175 6550 2175
+Wire Wire Line
+	6550 2175 6925 2175
 Wire Wire Line
 	7350 4850 7350 4700
@@
 	7025 1600 7025 1200
 Wire Wire Line
-	3350 2175 4325 2175
+	3350 2175 3475 2175
+Wire Wire Line
+	3475 2175 3875 2175
+Wire Wire Line
+	3875 2175 4100 2175
+Wire Wire Line
+	4100 2175 4325 2175
 Wire Wire Line
 	3875 2175 3875 2000
-Wire Wire Line
-	6000 3600 6000 3450
 Wire Wire Line
 	6425 1200 5700 1200
@@
 	6000 2375 6000 2650
 Wire Wire Line
-	6900 4400 6000 4400
+	6900 4400 5800 4400
 Wire Wire Line
 	4100 2075 4100 2175
@@
 Connection ~ 3475 2175
 Connection ~ 3350 2775
-Wire Wire Line
-	5800 3450 5500 3450
 $Comp
 L SA SA1
@@
 Connection ~ 6550 2175
 $Comp
-L POWER_GND #?
+L POWER_GND #011
 U 1 1 5315E6C5
-P 6550 3075
-F 0 "#?" V 6500 3025 60  0001 C CNN
-F 1 "POWER_GND" V 6600 3025 60  0001 C CNN
-F 2 "" H 6550 3075 60  0000 C CNN
-F 3 "" H 6550 3075 60  0000 C CNN
-	1    6550 3075
-	1    0    0    -1
-$EndComp
-Wire Wire Line
-	6550 3075 6550 2975
+P 6550 3675
+F 0 "#011" V 6500 3625 60  0001 C CNN
+F 1 "POWER_GND" V 6600 3625 60  0001 C CNN
+F 2 "" H 6550 3675 60  0000 C CNN
+F 3 "" H 6550 3675 60  0000 C CNN
+	1    6550 3675
+	1    0    0    -1
+$EndComp
+Wire Wire Line
+	6550 3675 6550 3450
+Wire Wire Line
+	6550 3450 6550 2975
+Wire Wire Line
+	6000 3450 6550 3450
+Connection ~ 6550 3450
+Wire Wire Line
+	5800 3600 5800 3600
+Wire Wire Line
+	5800 3600 5800 3450
 $EndSCHEMATC

Commit message: small changes
Parts:
- added XS3: питание радиомодуля, symbol CONN_02_F
- R1: value 5,1к -> 3,6к
Connections:
- net GND: now also XS3.2
- net V+: now also XS3.1
Changed lines of the file:
@@
 Sheet 1 1
 Title ""
-Date "8 mar 2014"
+Date "10 mar 2014"
 Rev ""
 Comp ""
@@
 P 5800 4400
 F 0 "R1" V 6350 4575 60  0000 C CNN
-F 1 "5,1к" V 6200 4175 60  0000 C CNN
+F 1 "3,6к" V 6200 4175 60  0000 C CNN
 F 2 "" H 5800 4400 60  0000 C CNN
 F 3 "" H 5800 4400 60  0000 C CNN
@@
 $EndComp
 Wire Wire Line
-	3150 2775 3350 2775
-Wire Wire Line
-	3350 2775 4275 2775
-Wire Wire Line
-	4275 2775 4325 2775
+	3150 2775 4325 2775
 Wire Wire Line
 	5325 2775 5450 2775
 Wire Wire Line
-	5325 2175 6550 2175
-Wire Wire Line
-	6550 2175 6925 2175
+	5325 2175 6925 2175
 Wire Wire Line
 	7350 4850 7350 4700
@@
 	7025 1600 7025 1200
 Wire Wire Line
-	3350 2175 3475 2175
-Wire Wire Line
-	3475 2175 3875 2175
-Wire Wire Line
-	3875 2175 4100 2175
-Wire Wire Line
-	4100 2175 4325 2175
+	3350 2175 4325 2175
 Wire Wire Line
 	3875 2175 3875 2000
@@
 	3350 2775 3350 2375
 Wire Wire Line
-	3475 3075 3475 2175
+	3475 1700 3475 3075
 Wire Wire Line
 	3350 2175 3350 2275
@@
 $EndComp
 Wire Wire Line
-	6550 3675 6550 3450
-Wire Wire Line
-	6550 3450 6550 2975
+	6550 2975 6550 3675
 Wire Wire Line
 	6000 3450 6550 3450
@@
 Wire Wire Line
 	5800 3600 5800 3450
+$Comp
+L CONN_02_F XS3
+U 1 1 531E09E3
+P 3325 1700
+F 0 "XS3" H 3575 1800 60  0000 C CNN
+F 1 "питание радиомодуля" H 3675 1500 60  0000 C CNN
+F 2 "" H 3325 1700 60  0000 C CNN
+F 3 "" H 3325 1700 60  0000 C CNN
+	1    3325 1700
+	-1   0    0    -1
+$EndComp
+Wire Wire Line
+	3325 1700 3475 1700
+Wire Wire Line
+	3325 1800 3600 1800
+Wire Wire Line
+	3600 1800 3600 2775
+Connection ~ 3600 2775
 $EndSCHEMATC
